Commit message: [version] Include depth cam in Sawyer URDF

File: sawyer_description/urdf/sawyer.urdf.xacro (robot description, xacro)
@@ -2,7 +2,8 @@
 <robot name="sawyer" xmlns:xacro="http://www.ros.org/wiki/xacro">
   <xacro:arg name="gazebo" default="false"/>
-  <xacro:arg name="pedestal" default="true"/>
+  <xacro:arg name="pedestal" default="false"/>
   <xacro:arg name="static" default="true"/>
   <xacro:arg name="electric_gripper" default="false"/>
+  <xacro:arg name="camera" default="true"/>
   <!-- Sawyer Base URDF -->
   <xacro:include filename="$(find sawyer_description)/urdf/sawyer_base.urdf.xacro">
@@ -22,3 +23,16 @@
   </xacro:include>
   </xacro:if>
+  <!-- Depth Camera -->
+  <xacro:if value="$(arg camera)">
+  <xacro:include filename="$(find realsense2_description)/urdf/_d435.urdf.xacro"/>
+  <xacro:sensor_d435 name="camera" parent="right_hand" use_nominal_extrinsics="true">
+    <origin xyz="0 -0.075 0.09" rpy="0 ${-pi/2} ${pi/2}"/>
+  </xacro:sensor_d435>
+  </xacro:if>
+<!--   <xacro:if value="$(arg camera)">
+  <xacro:include filename="$(find realsense2_description)/urdf/_d435.urdf.xacro"/>
+  <xacro:sensor_d435 name="camera" parent="head" use_nominal_extrinsics="true">
+    <origin xyz="0 0 0.45" rpy="0 ${pi/6} 0"/>
+  </xacro:sensor_d435>
+  </xacro:if> -->
 </robot>

File: sawyer_description/urdf/sawyer_base.urdf.xacro (robot description, xacro)
@@ -29,11 +29,11 @@
       </material>
     </visual>
-<xacro:unless value="$(arg gazebo)">
-    <inertial>
-      <origin rpy="0 0 0" xyz="0.000000 0.000000 0.000000"/>
-      <mass value="0.0001"/>
-      <inertia ixx="1e-08" ixy="0" ixz="0" iyy="1e-08" iyz="0" izz="1e-08"/>
-    </inertial>
-</xacro:unless>
+    <xacro:unless value="$(arg gazebo)">
+        <inertial>
+          <origin rpy="0 0 0" xyz="0.000000 0.000000 0.000000"/>
+          <mass value="0.0001"/>
+          <inertia ixx="1e-08" ixy="0" ixz="0" iyy="1e-08" iyz="0" izz="1e-08"/>
+        </inertial>
+    </xacro:unless>
   </link>
 <xacro:if value="$(arg pedestal)">
@@ -399,6 +399,6 @@
     <child link="right_l6"/>
     <axis xyz="0 0 1"/>
-<xacro:if value="$(arg gazebo)">
     <limit effort="9.0" lower="-3.14" upper="3.14" velocity="4.545"/>
+<xacro:if value="$(arg gazebo)">
     <dynamics damping="1.0" friction="0.5"/>
 </xacro:if>

Commit message: [ver] URDF camera pose update

File: sawyer_description/urdf/sawyer.urdf.xacro (robot description, xacro)
@@ -27,5 +27,5 @@
   <xacro:include filename="$(find sawyer_description)/urdf/_d435_mod.urdf.xacro"/>
   <xacro:sensor_d435 name="camera" parent="right_hand" use_nominal_extrinsics="true" gazebo="$(arg gazebo)">
-    <origin xyz="0 -0.075 0.09" rpy="0 ${-pi/2} ${pi/2}"/>
+    <origin xyz="0 -0.07 0.07" rpy="0 ${-pi/2} ${pi/2}"/>
   </xacro:sensor_d435>
   </xacro:if>

Commit message: Gripper Hand3 mesh included

File: sawyer_description/urdf/sawyer.urdf.xacro (robot description, xacro)
@@ -40,19 +40,19 @@
   <link name="bigass_gripper">
     <visual>
-      <origin rpy="0 0 0" xyz="0 0 0.125"/>
+      <origin rpy="3.14 0 1.57" xyz="-0.035 0 -0.14"/>
+      <geometry>
+        <mesh filename="package://sawyer_description/meshes/rtlions_hand3/GripperCaseFix_v1.stl" scale="0.0008 0.001 0.00107"/>
+      </geometry>
+      <material name="sawyer_gray"/>
+    </visual>
+    <collision>
+      <origin rpy="0 0 0" xyz="0 0 -0.09"/>
       <geometry>
         <box size="0.10 0.15 0.2"/>
-      </geometry>
-      <material name="darkgray"/>
-    </visual>
-    <collision>
-      <origin rpy="0 0 0" xyz="0 0 0.125"/>
-      <geometry>
-        <box size="0.2 0.2 0.25"/>
       </geometry>
     </collision>
   </link>
   <joint name="gripper_joint" type="fixed">
-    <origin rpy="0 0 0" xyz="0.0 0.0 0.03"/>
+    <origin rpy="0 0 0" xyz="0.05 0.0 0.21"/>
     <parent link="right_hand"/>
     <child link="bigass_gripper"/>
